Commit message: 修改u_shaped_gimbal为u_shaped_gimbal_description，以符合规范

File: v2/u_shaped_gimbal_description/urdf/u_shaped_gimbal.urdf (robot description, URDF)
Before this commit: robot u_shaped_gimbal, 5 links, 4 joints
Links:
- link base_link: geometry collision mesh filename=package://u_shaped_gimbal_description/meshes/base_link.STL; visual mesh filename=package://u_shaped_gimbal_description/meshes/base_link.STL
- link link_front: geometry collision mesh filename=package://u_shaped_gimbal_description/meshes/link_front.STL; visual mesh filename=package://u_shaped_gimbal_description/meshes/link_front.STL
- link link_low: geometry collision mesh filename=package://u_shaped_gimbal_description/meshes/link_low.STL; visual mesh filename=package://u_shaped_gimbal_description/meshes/link_low.STL
- link link_middle: geometry collision mesh filename=package://u_shaped_gimbal_description/meshes/link_middle.STL; visual mesh filename=package://u_shaped_gimbal_description/meshes/link_middle.STL
- link link_up: geometry collision mesh filename=package://u_shaped_gimbal_description/meshes/link_up.STL; visual mesh filename=package://u_shaped_gimbal_description/meshes/link_up.STL

Commit message: 将云台放正

File: v2/u_shaped_gimbal_description/urdf/u_shaped_gimbal.urdf (robot description, URDF)
Before this commit: robot u_shaped_gimbal, 5 links, 4 joints
Links:
- added link root_link
Joints:
- added joint root_to_base: type fixed, parent root_link, child base_link, origin xyz=0 0 0 rpy=1.5708 0 1.5708
